File: traffic-lights.kicad_sch (KiCad schematic)
At the start: 7 parts, among them J1 uPMOD

Commit message: add readme
Parts:
- R1, R2, R3: value 470R -> 200R
Changed lines of the file:
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@@
       (effects (font (size 1.27 1.27)))
     )
-    (property "Value" "470R" (at 74.93 92.71 90)
+    (property "Value" "200R" (at 74.93 92.71 90)
       (effects (font (size 1.27 1.27)))
     )
@@
       (effects (font (size 1.27 1.27)))
     )
-    (property "Value" "470R" (at 74.93 97.79 90)
+    (property "Value" "200R" (at 74.93 97.79 90)
       (effects (font (size 1.27 1.27)))
     )
@@
       (effects (font (size 1.27 1.27)))
     )
-    (property "Value" "470R" (at 74.93 95.25 90)
+    (property "Value" "200R" (at 74.93 95.25 90)
       (effects (font (size 1.27 1.27)))
     )
